File: Projects/EagleProjects/Tranciver/Schematic.sch (EAGLE design)
At the start: 29 parts, among them IC1 LM317MBSTT3, IC2 AD8597R, Q1 2N7000G, U1 ADA4091-2ARZ-RL, U2 TC4427AEOA

Commit message: schmatic for eagle
Parts:
- added R12, R13, R17: (no value), resistor:R-US_M0805
- added R14, R16: (no value), pot:TRIM_EU-CA6V
- R11: device pot-vitrohm:PC25 -> pot:TRIM_EU-CA6V
Connections:
- removed net N$11: C7.2, IC2.+VS
- removed net N$15: R7.2
- removed net N$8: C5.2, U1.V+
- new net N$16: R13.2, R17.1, U1.INA-
- new net N$18: R12.1, R5.2, U$1.A22/DAC1
- new net N$19: R14.S
- new net N$21: R11.S, R13.1
- new net N$22: R14.A, R17.2
- net GND: now also R11.E, R12.2
- net N$10: now also R16.S; no longer R11.S
- net N$13: now also R16.A; no longer R11.A
- net N$14: now also R16.E; no longer R11.E
- net N$17: now also R5.1; no longer U1.INA-
- net VO: now also C5.2, C7.2, IC2.+VS, R7.2, U1.V+
Other:
- moved on the sheet: C1, C2, C3, D1, D2, IC1, R1, R2, R5
