File: Projects/EagleProjects/Tranciver/Transiver_Schematic.sch (EAGLE design)
At the start: 14 parts, among them IC1 LM317MBSTT3, Q1 2N7000G, U1 ADA4091-2ARZ-RL, U2 TC4427AEOA, U3 ADA4091-2ARZ-RL

Commit message: eagle work
Parts:
- removed Q1: 2N7000G, 2N7000G:2N7000G
- removed SP1: MA40S4S, Parts:MA40S4S
- removed U1: ADA4091-2ARZ-RL, ADA4091-2ARZ-RL:ADA4091-2ARZ-RL
- removed U2: TC4427AEOA, Parts:TC4427AEOA
- added C12, C13, C14, C15, C16: 100nF, capacitor-wima:C2,5-3
- added D7: 3V3, diode:1N4728
- added IC4: AD8597R, analog-devices:AD8597R
- added J1: 18V, 694102303002:694102303002
- added Q2: 2N7000G, 2N7000G:2N7000G
- added R22, R23, R31, R32, R34, R35: (no value), resistor:R-US_M0805
- added R24, R30, R33: (no value), pot:TRIM_EU-CA6V
- added R25: 10k, resistor:R-US_R0805
- added R26, R28, R29: 100, resistor:R-US_M0805
- added R27: 1M, resistor:R-US_M0805
- added SP2: MA40S4S, Parts:MA40S4S
- added U4: ADA4091-2ARZ-RL, ADA4091-2ARZ-RL:ADA4091-2ARZ-RL
- U3: value ADA4091-2ARZ-RL -> TC4427AEOA; device ADA4091-2ARZ-RL:ADA4091-2ARZ-RL -> Parts:TC4427AEOA
Connections:
- removed net N$2: U$1.2, U2.IN_A
- removed net VIN: C1.1, D1.C, IC1.IN
- removed net VO: C2.+, D1.A, D2.C, IC1.OUT, R1.2
- new net 12V: C12.2, C15.2, IC4.+VS, U4.V+
- new net 18V: C1.1, D1.C, IC1.IN, J1.1
- new net A0: R34.2, R35.1, U$1.14/A0
- new net D5: U$1.5, U3.IN_A
- new net D7: R26.1, R27.1, U$1.7
- new net N$23: IC4.IN+, R24.S
- new net N$24: D7.C, R23.1, R24.E
- new net N$25: R22.1, R24.A
- new net N$27: R28.2, R29.2, U4.INA+
- new net N$28: C14.2, U3.VDD
- new net N$30: R25.2, SP2.1, U3.*OUT_A
- new net N$31: Q2.GATE, R26.2
- new net N$33: R31.2, R32.1, U4.INA-
- new net N$34: R30.S, R34.1, U4.OUTA
- new net N$36: R31.1, R33.S
- new net N$37: R30.A, R32.2
- new net OPAMP: Q2.DRN, Q2.SRC, R25.1, R27.2, R28.1, SP2.2
- new net VDD: C2.+, D1.A, D2.C, IC1.OUT, R1.2, R23.2
- new net VREF: IC4.OUT, R29.1
- net GND: now also C12.1, C13.1, C13.2, C14.1, C15.1, C16.1, C16.2, D7.A, IC4.-VS, J1.2, R22.2, R33.E, R35.2, U$1.AGND, U3.GND, U4.V-; no longer U2.GND
Other:
- note added: "OP-AMP Circuit"
- note added: "Transceiver"
- note added: "Voltage Reference"
- note removed: "12V, 500mA"
- note removed: "3V - 40V DC"
- moved on the sheet: C1, C2, C3, D1, D2, IC1, R1, R2, U3
